Commit message: Decouple two joints movement

File: mnlm/robot/robot_arm_ws/src/robot_arm/models/arm.urdf (robot description, URDF)
Before this commit: robot robot_arm, 3 links, 2 joints
Joints:
- joint servo1: axis 0 1 0 -> 0 0 1

Commit message: update

File: mnlm/robot/robot_arm_ws/src/robot_arm/models/arm.urdf (robot description, URDF)
Before this commit: robot robot_arm, 3 links, 2 joints
Links:
- added link dummy_lower_body_link, mass 1.0; collision box size=0.4 0.4 0.4; visual box size=0.4 0.4 0.4
- link lower_body: geometry collision cylinder length=1.0 radius=0.25; visual cylinder length=1.0 radius=0.25
Joints:
- added joint dummy_lower_body_joint: type revolute, parent dummy_lower_body_link, child upper_body, origin xyz=-0.5 0 0.4 rpy=0 0 0, limit lower=0.0 upper=1.57 effort=1000 velocity=10.0
- joint servo1: axis 0 0 1 -> 0 1 0; child upper_body -> dummy_lower_body_link; limit lower=-1.57 upper=1.57 effort=1000 velocity=1.0 -> lower=0.0 upper=1.57 effort=1000 velocity=1.0; origin xyz=0 0 0.45 rpy=0 0 0 -> xyz=0 0 0.7 rpy=0 0 0

Commit message: middle body rotate in the good position, but friction too high

File: mnlm/robot/robot_arm_ws/src/robot_arm/models/arm.urdf (robot description, URDF)
Before this commit: robot robot_arm, 3 links, 2 joints
Links:
- removed link dummy_lower_body_link
- added link middle_body, mass 1.0; collision box size=0.3 0.3 1.4; visual box size=0.3 0.3 1.4
- added link world
Joints:
- added joint base_joint: type fixed, parent world, child base, origin xyz=1.5 1.0 0 rpy=0 0 0
- joint servo1: child dummy_lower_body_link -> middle_body; origin xyz=0 0 0 rpy=0 0 0 -> xyz=0 0 0.5 rpy=0 0 0

Commit message: Adjusted the velocity and inertia, moving more naturally

File: mnlm/robot/robot_arm_ws/src/robot_arm/models/arm.urdf (robot description, URDF)
Before this commit: robot robot_arm, 4 links, 3 joints
Joints:
- joint servo0: limit lower=-1.57 upper=1.57 effort=10000 velocity=1.0 -> lower=-1.57 upper=1.57 effort=1000 velocity=2.0
- joint servo1: limit lower=0.0 upper=1.57 effort=10000 velocity=1.0 -> lower=-1.57 upper=1.57 effort=1000 velocity=2.0

Commit message: Add more joints

File: mnlm/robot/robot_arm_ws/src/robot_arm/models/arm.urdf (robot description, URDF)
Before this commit: robot robot_arm, 4 links, 3 joints
Links:
- added link upper_middle_body, mass 1.0; collision box size=0.3 0.3 1.0; visual box size=0.3 0.3 1.0
- link middle_body: geometry collision box size=0.3 0.3 1.2; visual box size=0.3 0.3 1.2
Joints:
- added joint servo2: type revolute, parent middle_body, child upper_middle_body, origin xyz=0 0 0.9 rpy=0 0 0, axis 0 1 0, limit lower=-1.57 upper=1.57 effort=1000 velocity=2.0

Commit message: Add the upper body

File: mnlm/robot/robot_arm_ws/src/robot_arm/models/arm.urdf (robot description, URDF)
Before this commit: robot robot_arm, 5 links, 4 joints
Links:
- added link upper_body, mass 1.0; collision box size=0.3 0.3 0.8; visual box size=0.3 0.3 0.8
Joints:
- added joint servo3: type revolute, parent upper_middle_body, child upper_body, origin xyz=0 0 1.0 rpy=0 0 0, axis 0 1 0, limit lower=-1.57 upper=1.57 effort=1000 velocity=2.0

Commit message: Use arm.xacro instead of arm.urdf

File: mnlm/robot/robot_arm_ws/src/robot_arm/models/arm.urdf (robot description, URDF)
Before this commit: robot robot_arm, 6 links, 5 joints
Links:
- added link gripper_base, mass 1.0; collision box size=0.5 0.5 0.1; visual box size=0.5 0.5 0.1
Joints:
- added joint servo4: type revolute, parent upper_body, child gripper_base, origin xyz=0 0 0.45 rpy=0 0 0, axis 0 0 1, limit lower=-1.57 upper=1.57 effort=1000 velocity=2.0

File: mnlm/robot/robot_arm_ws/src/robot_arm/models/arm.xacro (robot description, xacro)
@@ -1,8 +1,5 @@
 <?xml version="1.0"?>
 <robot xmlns:xacro="http://www.ros.org/wiki/xacro" name="robot_arm">
-    <!-- This first link called "world" is empty -->
     <link name="world"></link>
-    <!-- A simple fixed joint from our empty world link, to our base. -->
-    <!-- The base origin is offset from the world origin. -->
     <joint name="base_joint" type="fixed">
         <origin xyz="1.5 1.0 0" rpy="0 0 0"/>
@@ -26,5 +23,5 @@
         <inertial>
             <mass value="1.0"/>
-            <inertia ixx="1" ixy="0" ixz="0" iyy="1" iyz="0" izz="1"/>
+            <inertia ixx="0.001" ixy="0" ixz="0" iyy="0.001" iyz="0" izz="0.001"/>
         </inertial>
     </link>
@@ -45,5 +42,6 @@
         <inertial>
             <mass value="1.0"/>
-            <inertia ixx="0.034375" ixy="0" ixz="0" iyy="0.034375" iyz="0" izz="0.0171875"/>
+            <!-- Inertia tensor for a cylinder with mass=1kg, radius=0.25, and length=0.5 -->
+            <inertia ixx="0.0001" ixy="0" ixz="0" iyy="0.0001" iyz="0" izz="0.0001"/>
         </inertial>
     </link>
@@ -53,11 +51,11 @@
         <origin xyz="0.5 0 0.5" rpy="0 0 0"/>
         <axis xyz="0 0 1"/>
-        <limit lower="-1.57" upper="1.57" effort="10000" velocity="1.0"/>
-    </joint>
-    <link name="dummy_lower_body_link">
-        <visual>
-            <origin xyz="0 0 1.2" rpy="0 0 0"/>
-            <geometry>
-                <box size="0.4 0.4 1.4"/>
+        <limit lower="-1.57" upper="1.57" effort="1000" velocity="2.0"/>
+    </joint>
+    <link name="middle_body">
+        <visual>
+            <origin xyz="0 0 0.5" rpy="0 0 0"/>
+            <geometry>
+                <box size="0.3 0.3 1.2"/>
             </geometry>
             <material name="grey">
@@ -66,45 +64,104 @@
         </visual>
         <collision>
-            <origin xyz="0 0 1.2" rpy="0 0 0"/>
-            <geometry>
-                <box size="0.4 0.4 0.4"/>
-            </geometry>
-        </collision>
-        <inertial>
-            <mass value="1.0"/>
-            <inertia ixx="1e-6" ixy="0" ixz="0" iyy="1e-6" iyz="0" izz="1e-6"/>
+            <origin xyz="0 0 0.5" rpy="0 0 0"/>
+            <geometry>
+                <box size="0.3 0.3 1.2"/>
+            </geometry>
+        </collision>
+        <inertial>
+            <mass value="1.0"/>
+            <inertia ixx="0.000117" ixy="0" ixz="0" iyy="0.000117" iyz="0" izz="0.0000117"/>
         </inertial>
     </link>
     <joint name="servo1" type="revolute">
         <parent link="lower_body"/>
-        <child link="dummy_lower_body_link"/>
-        <origin xyz="0.5 0 0" rpy="0 0 0"/>
+        <child link="middle_body"/>
+        <origin xyz="0 0 0.5" rpy="0 0 0"/>
         <axis xyz="0 -1 0"/>
-        <limit lower="0.0" upper="1.57" effort="10000" velocity="1.0"/>
+        <limit lower="-1.57" upper="1.57" effort="1000" velocity="2.0"/>
+    </joint>
+    <link name="upper_middle_body">
+        <visual>
+            <origin xyz="0 0 0.6" rpy="0 0 0"/>
+            <geometry>
+                <box size="0.3 0.3 1.0"/>
+            </geometry>
+            <material name="dark_green">
+                <color rgba="0.5 0.5 0.5 1"/>
+            </material>
+        </visual>
+        <collision>
+            <origin xyz="0 0 0.6" rpy="0 0 0"/>
+            <geometry>
+                <box size="0.3 0.3 1.0"/>
+            </geometry>
+        </collision>
+        <inertial>
+            <mass value="1.0"/>
+            <inertia ixx="0.000117" ixy="0" ixz="0" iyy="0.000117" iyz="0" izz="0.0000117"/>
+        </inertial>
+    </link>
+    <joint name="servo2" type="revolute">
+        <parent link="middle_body"/>
+        <child link="upper_middle_body"/>
+        <origin xyz="0 0 0.9" rpy="0 0 0"/>
+        <axis xyz="0 1 0"/>
+        <limit lower="-1.57" upper="1.57" effort="1000" velocity="2.0"/>
     </joint>
     <link name="upper_body">
         <visual>
-            <geometry>
-                <box size="1.4 0.4 0.4"/>
+            <origin xyz="0 0 0.4" rpy="0 0 0"/>
+            <geometry>
+                <box size="0.3 0.3 0.8"/>
+            </geometry>
+            <material name="black">
+                <color rgba="0.5 0.5 0.5 1"/>
+            </material>
+        </visual>
+        <collision>
+            <origin xyz="0 0 0.4" rpy="0 0 0"/>
+            <geometry>
+                <box size="0.3 0.3 0.8"/>
+            </geometry>
+        </collision>
+        <inertial>
+            <mass value="1.0"/>
+            <inertia ixx="0.000117" ixy="0" ixz="0" iyy="0.000117" iyz="0" izz="0.0000117"/>
+        </inertial>
+    </link>
+    <joint name="servo3" type="revolute">
+        <parent link="upper_middle_body"/>
+        <child link="upper_body"/>
+        <origin xyz="0 0 1.0" rpy="0 0 0"/>
+        <axis xyz="0 1 0"/>
+        <limit lower="-1.57" upper="1.57" effort="1000" velocity="2.0"/>
+    </joint>
+    <link name="gripper_base">
+        <visual>
+            <origin xyz="0 0 0.4" rpy="0 0 0"/>
+            <geometry>
+                <box size="0.5 0.5 0.1"/>
             </geometry>
             <material name="dark_green">
-                <color rgba="0.5 0.5 1.0 1"/>
-            </material>
-        </visual>
-        <collision>
-            <geometry>
-                <box size="1.4 0.4 0.4"/>
-            </geometry>
-        </collision>
-        <inertial>
-            <mass value="0.1"/>
-            <inertia ixx="1e-6" ixy="0" ixz="0" iyy="1e-6" iyz="0" izz="1e-6"/>
-        </inertial>
-    </link>
-    <joint name="dummy_lower_body_joint" type="fixed">
-        <parent link="dummy_lower_body_link"/>
-        <child link="upper_body"/>
-        <origin xyz="-0.2 0 0.4" rpy="0 0 0"/>
-        <axis xyz="0 1 0"/>
+                <color rgba="0 0 0 1"/>
+            </material>
+        </visual>
+        <collision>
+            <origin xyz="0 0 0.4" rpy="0 0 0"/>
+            <geometry>
+                <box size="0.5 0.5 0.1"/>
+            </geometry>
+        </collision>
+        <inertial>
+            <mass value="1.0"/>
+            <inertia ixx="0.000117" ixy="0" ixz="0" iyy="0.000117" iyz="0" izz="0.0000117"/>
+        </inertial>
+    </link>
+    <joint name="servo4" type="revolute">
+        <parent link="upper_body"/>
+        <child link="gripper_base"/>
+        <origin xyz="0 0 0.45" rpy="0 0 0"/>
+        <axis xyz="0 0 1"/>
+        <limit lower="-1.57" upper="1.57" effort="1000" velocity="2.0"/>
     </joint>
     <gazebo>
@@ -123,4 +180,5 @@
             <state_interface name="position"/>
             <state_interface name="velocity"/>
+            <!-- <state_interface name="effort"/> -->
         </joint>
         <joint name="servo1">
@@ -128,4 +186,23 @@
             <state_interface name="position"/>
             <state_interface name="velocity"/>
+            <!-- <state_interface name="effort"/> -->
+        </joint>
+        <joint name="servo2">
+            <command_interface name="position"/>
+            <state_interface name="position"/>
+            <state_interface name="velocity"/>
+            <!-- <state_interface name="effort"/> -->
+        </joint>
+        <joint name="servo3">
+            <command_interface name="position"/>
+            <state_interface name="position"/>
+            <state_interface name="velocity"/>
+            <!-- <state_interface name="effort"/> -->
+        </joint>
+        <joint name="servo4">
+            <command_interface name="position"/>
+            <state_interface name="position"/>
+            <state_interface name="velocity"/>
+            <!-- <state_interface name="effort"/> -->
         </joint>
     </ros2_control>
