Commit message: A working version, but the rotate point of upper_body is off

File: mnlm/robot/robot_arm_ws/src/robot_arm/models/arm.xacro (robot description, xacro)
@@ -1,10 +1,13 @@
 <?xml version="1.0"?>
-<robot name="robot_arm">
-    <!-- <link name="world"></link>
+<robot xmlns:xacro="http://www.ros.org/wiki/xacro" name="robot_arm">
+    <!-- This first link called "world" is empty -->
+    <link name="world"></link>
+    <!-- A simple fixed joint from our empty world link, to our base. -->
+    <!-- The base origin is offset from the world origin. -->
     <joint name="base_joint" type="fixed">
         <origin xyz="1.5 1.0 0" rpy="0 0 0"/>
         <parent link="world"/>
         <child link="base"/>
-    </joint> -->
+    </joint>
     <link name="base">
         <visual>
@@ -42,5 +45,4 @@
         <inertial>
             <mass value="1.0"/>
-            <!-- Inertia tensor for a cylinder with mass=1kg, radius=0.25, and length=0.5 -->
             <inertia ixx="0.034375" ixy="0" ixz="0" iyy="0.034375" iyz="0" izz="0.0171875"/>
         </inertial>
@@ -77,9 +79,9 @@
         <parent link="lower_body"/>
         <child link="dummy_lower_body_link"/>
-        <origin xyz="0 0 0" rpy="0 0 0"/>
+        <origin xyz="0.5 0 0" rpy="0 0 0"/>
         <axis xyz="0 -1 0"/>
         <limit lower="0.0" upper="1.57" effort="10000" velocity="1.0"/>
     </joint>
-    <!-- <link name="upper_body">
+    <link name="upper_body">
         <visual>
             <geometry>
@@ -105,5 +107,5 @@
         <origin xyz="-0.2 0 0.4" rpy="0 0 0"/>
         <axis xyz="0 1 0"/>
-</joint> -->
+    </joint>
     <gazebo>
         <plugin filename="/opt/ros/humble/lib/libign_ros2_control-system.so" name="ign_ros2_control::IgnitionROS2ControlPlugin">
@@ -121,5 +123,4 @@
             <state_interface name="position"/>
             <state_interface name="velocity"/>
-            <!-- <state_interface name="effort"/> -->
         </joint>
         <joint name="servo1">
@@ -127,5 +128,4 @@
             <state_interface name="position"/>
             <state_interface name="velocity"/>
-            <!-- <state_interface name="effort"/> -->
         </joint>
     </ros2_control>

Commit message: complete arm

File: mnlm/robot/robot_arm_ws/src/robot_arm/models/arm.xacro (robot description, xacro)
@@ -137,5 +137,5 @@
         <limit lower="-1.57" upper="1.57" effort="1000" velocity="2.0"/>
     </joint>
-    <link name="gripper_base">
+    <link name="top_link">
         <visual>
             <origin xyz="0 0 0.4" rpy="0 0 0"/>
@@ -160,8 +160,64 @@
     <joint name="servo4" type="revolute">
         <parent link="upper_body"/>
-        <child link="gripper_base"/>
+        <child link="top_link"/>
         <origin xyz="0 0 0.45" rpy="0 0 0"/>
         <axis xyz="0 0 1"/>
         <limit lower="-1.57" upper="1.57" effort="1000" velocity="2.0"/>
+    </joint>
+    <link name="gripper_left_finger">
+        <visual>
+            <origin xyz="0 0 0.1" rpy="0 0 0"/>
+            <geometry>
+                <box size="0.1 0.1 0.4"/>
+            </geometry>
+            <material name="grey">
+                <color rgba="0 0 0 1"/>
+            </material>
+        </visual>
+        <collision>
+            <origin xyz="0 0 0.1" rpy="0 0 0"/>
+            <geometry>
+                <box size="0.1 0.1 0.4"/>
+            </geometry>
+        </collision>
+        <inertial>
+            <mass value="1.0"/>
+            <inertia ixx="0.000117" ixy="0" ixz="0" iyy="0.000117" iyz="0" izz="0.0000117"/>
+        </inertial>
+    </link>
+    <joint name="left_gripper_joint" type="prismatic">
+        <parent link="top_link"/>
+        <child link="gripper_left_finger"/>
+        <origin xyz="0 0.2 0.5" rpy="0 0 0"/>
+        <axis xyz="0 -1 0"/>
+        <limit lower="-0.3" upper="0.3" effort="100.0" velocity="1.0"/>
+    </joint>
+    <link name="gripper_right_finger">
+        <visual>
+            <origin xyz="0 0 0.1" rpy="0 0 0"/>
+            <geometry>
+                <box size="0.1 0.1 0.4"/>
+            </geometry>
+            <material name="dark_green">
+                <color rgba="0 0 0 1"/>
+            </material>
+        </visual>
+        <collision>
+            <origin xyz="0 0 0.1" rpy="0 0 0"/>
+            <geometry>
+                <box size="0.1 0.1 0.4"/>
+            </geometry>
+        </collision>
+        <inertial>
+            <mass value="1.0"/>
+            <inertia ixx="0.000117" ixy="0" ixz="0" iyy="0.000117" iyz="0" izz="0.0000117"/>
+        </inertial>
+    </link>
+    <joint name="right_gripper_joint" type="prismatic">
+        <parent link="top_link"/>
+        <child link="gripper_right_finger"/>
+        <origin xyz="0 -0.2 0.5" rpy="0 0 0"/>
+        <axis xyz="0 1 0"/>
+        <limit lower="-0.3" upper="0.3" effort="100.0" velocity="1.0"/>
     </joint>
     <gazebo>
@@ -206,4 +262,16 @@
             <!-- <state_interface name="effort"/> -->
         </joint>
+        <joint name="left_gripper_joint">
+            <command_interface name="position"/>
+            <state_interface name="position"/>
+            <state_interface name="velocity"/>
+            <!-- <state_interface name="effort"/> -->
+        </joint>
+        <joint name="right_gripper_joint">
+            <command_interface name="position"/>
+            <state_interface name="position"/>
+            <state_interface name="velocity"/>
+            <!-- <state_interface name="effort"/> -->
+        </joint>
     </ros2_control>
 </robot>

File: mnlm/robot/robot_arm_ws/src/robot_arm/models/gripper.xacro (robot description, xacro)
@@ -1,5 +1,15 @@
+<?xml version="1.0"?>
 <!--https://github.com/PacktPublishing/ROS-Robotics-By-Example/blob/master/Chapter_5_code/ros_robotics/urdf/gripper.xacro-->
-<?xml version="1.0"?>
-<robot xmlns:xacro="http://www.ros.org/wiki/xacro">
+<robot xmlns:xacro="http://www.ros.org/wiki/xacro" name="gripper">
+    <xacro:property name="height2" value="1" />
+    <xacro:property name="axle_offset" value="0.05" />
+    <!-- Default Inertial -->
+    <xacro:macro name="default_inertial" params="z_value i_value mass">
+        <inertial>
+            <origin xyz="0 0 ${z_value}" rpy="0 0 0"/>
+            <mass value="${mass}" />
+            <inertia ixx="${i_value}" ixy="0.0" ixz="0.0" iyy="${i_value}" iyz="0.0" izz="${i_value}" />
+        </inertial>
+    </xacro:macro>
     <!-- Gripper -->
     <joint name="left_gripper_joint" type="revolute">
@@ -14,5 +24,5 @@
             <origin rpy="0 0 0" xyz="0 0 0"/>
             <geometry>
-                <mesh filename="package://ros_robotics/meshes/l_finger.dae"/>
+                <mesh filename="$(find robot_arm)/meshes/l_finger.dae"/>
             </geometry>
         </visual>
@@ -32,5 +42,5 @@
             <origin rpy="0 0 0" xyz="0.09137 0.00495 0"/>
             <geometry>
-                <mesh filename="package://ros_robotics/meshes/l_finger_tip.dae"/>
+                <mesh filename="$(find robot_arm)/meshes/l_finger_tip.dae"/>
             </geometry>
         </visual>
@@ -53,5 +63,5 @@
             <origin rpy="3.1415 0 0" xyz="0 0 0"/>
             <geometry>
-                <mesh filename="package://ros_robotics/meshes/l_finger.dae"/>
+                <mesh filename="$(find robot_arm)/meshes/l_finger.dae"/>
             </geometry>
         </visual>
@@ -71,5 +81,5 @@
             <origin rpy="-3.1415 0 0" xyz="0.09137 0.00495 0"/>
             <geometry>
-                <mesh filename="package://ros_robotics/meshes/l_finger_tip.dae"/>
+                <mesh filename="$(find robot_arm)/meshes/l_finger_tip.dae"/>
             </geometry>
         </visual>
@@ -81,23 +91,3 @@
         <xacro:default_inertial z_value="0" i_value="1e-6" mass="1e-5"/>
     </link>
-    <transmission name="gripper_transmission1">
-        <type>transmission_interface/SimpleTransmission</type>
-        <joint name="left_gripper_joint">
-            <hardwareInterface>EffortJointInterface</hardwareInterface>
-        </joint>
-        <actuator name="gripper_motor1">
-            <hardwareInterface>EffortJointInterface</hardwareInterface>
-            <mechanicalReduction>1</mechanicalReduction>
-        </actuator>
-    </transmission>
-    <transmission name="gripper_transmission2">
-        <type>transmission_interface/SimpleTransmission</type>
-        <joint name="right_gripper_joint">
-            <hardwareInterface>EffortJointInterface</hardwareInterface>
-        </joint>
-        <actuator name="gripper_motor2">
-            <hardwareInterface>EffortJointInterface</hardwareInterface>
-            <mechanicalReduction>1</mechanicalReduction>
-        </actuator>
-    </transmission>
 </robot>
